File: DiodeCompressor/Analog.kicad_sch (KiCad schematic)
At the start: 54 parts, among them U1 TL074, U2 TL074, U3 TL074

Commit message: firmware boilerplate for MCU
Parts:
- added R31, R32, R33, R34, R36: 100k, Resistor_SMD:R_0805_2012Metric, symbol Device:R_US
- added R35: 22k, Resistor_SMD:R_0805_2012Metric, symbol Device:R_US
Connections:
- net AmpAnode: now also R31.1
- net FX_OUT: now also RV4.2; no longer C8.2, RV4.3
- net GND: now also R34.1, R36.1
- net VG: now also R32.1
- net at U3.5 (+): now also R32.2, R34.2
- net at U3.6 (-): now also R31.2, R33.1
- net at U3.7: now also R33.2, R35.2
- new net: C8.2, RV4.3
- new net vADC: R35.1, R36.2
Other:
- moved on the sheet: C1, C2, C4, C7, R1, R2, U1A, U1E, U2E, U3E
